Commit message: final saturday changes - mostly routine

File: src/astro_launch/urdf/rover.urdf (robot description, URDF)
Before this commit: robot simple_rover, 3 links, 2 joints
Links:
- removed link tag_link
- link base_link: geometry visual box size=1.38 0.74 0.61
Joints:
- removed joint tag_to_base
- joint camera_joint: origin xyz=0.4 0 0.2 rpy=0 0 0 -> xyz=0.52 0.0 0.44 rpy=0 0 0
